File: Connectors.kicad_sch (KiCad schematic)
At the start: 14 parts, among them J1 USB_B_Micro, J10 M20-9990246, J2 WE-RJ45_7499211123A, J21 Conn_02x18_Odd_Even, J22 Conn_02x18_Odd_Even

Commit message: BOM Finalization, board cleanup.
Parts:
- J1: Comment 10103594-0001LF -> C428495 10103594-0001LF
- J2: Comment 7499211123A -> C24363903 7499211123A; PART-NUMBER (none) -> C24363903
Changed lines of the file:
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@@
 			)
 		)
-		(property "PART-NUMBER" ""
+		(property "PART-NUMBER" "C24363903 "
 			(at 124.46 137.16 0)
 			(effects
@@
 			)
 		)
-		(property "Comment" "7499211123A"
+		(property "Comment" "C24363903 7499211123A"
 			(at 124.46 137.16 0)
 			(effects
@@
 			)
 		)
-		(property "Comment" "10103594-0001LF"
+		(property "Comment" "C428495 10103594-0001LF"
 			(at 115.57 40.64 0)
 			(effects
