File: POEPico.kicad_pcb (KiCad board)
At the start: 4 copper layers, 40 x 100 mm, 142 parts, among them J1 USB_B_Micro, J10 M20-9990246, J2 WE-RJ45_7499211123A, J21 Conn_02x18_Odd_Even, J22 Conn_02x18_Odd_Even, Q1 PSMN075-100MSEX, Q10 FMMT723QTA, Q11 BSZ900N20NS3GATMA1, Q12 TPN1600ANH, Q13 MMBT3906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

Commit message: BOM Cleanup and matching for JLCPCB, downstream edits to Schematic and Board. Added backup files to .gitignore.
Parts:
- D5: value BAS19LT1G -> BAS21_R1_00001
- R1, R11, R12, R13, R14, R15, R16, R17, R18, R19, R2, R20, R3, R31, R32, R33, R5: footprint Capacitor_SMD:C_0402_1005Metric -> Resistor_SMD:R_0402_1005Metric
- R10, R21, R22, R23, R24, R25, R29, R30, R34, R36, R6, R7, R9: footprint Capacitor_SMD:C_0603_1608Metric -> Resistor_SMD:R_0603_1608Metric
- R26: footprint Capacitor_SMD:C_0805_2012Metric -> Resistor_SMD:R_0805_2012Metric
- R27: footprint LED_SMD:LED_0805_2012Metric -> Resistor_SMD:R_0805_2012Metric
- R28: footprint Capacitor_SMD:C_0805_2012Metric -> Resistor_SMD:R_1210_3225Metric
- R4: footprint Diode_SMD:D_0402_1005Metric -> Resistor_SMD:R_0402_1005Metric
- moved R28 0.92 mm to (145.0, 68.9)
Routing:
- net Net-(C50-Pad2): track 1.78 -> 3.79 mm
- net Net-(R24-Pad1): track 33.7 -> 35.1 mm, vias 0 -> 2
- net Net-(U3-VIN): track 79.9 -> 79.0 mm, vias 3 -> 2

Commit message: BOM Finalization, board cleanup.
Parts:
- D4: value PTVS58VP1UTP -> SMF58A; footprint Diode_SMD:D_SOD-128 -> Diode_SMD:D_SOD-123
- L1: footprint Custom:DO1608C -> Custom:FCH5030-100M
- L3: footprint Custom:DO1608C -> Custom:AABG05A20M101
- L4: footprint Custom:DO1813H -> Inductor_SMD:L_0603_1608Metric
- moved L1 3.30 mm to (141.7, 32.6)
- moved L4 3.24 mm to (126.4, 87.1)
- moved L3 3.17 mm to (138.5, 46.9)
- moved R21 1.31 mm to (140.5, 30.9)
- moved D4 1.30 mm to (137.8, 30.0)
Routing:
- net Net-(U3-HSSRC): track 8.24 -> 11.4 mm
- net +12V0: track 107.4 -> 110.0 mm
- net Net-(C46-Pad1): track 35.9 -> 38.4 mm
- net VSS: track 135.3 -> 136.8 mm
- net Net-(U3-VPORT): track 4.43 -> 5.67 mm
- net Net-(C44-Pad1): track 34.5 -> 33.5 mm
