File: Power.kicad_sch (KiCad schematic)
At the start: 72 parts, among them Q1 PSMN075-100MSEX, Q10 FMMT723QTA, Q11 BSZ900N20NS3GATMA1, Q12 TPN1600ANH, Q13 MMBT3906, Q14 MMBT3904, Q2 PSMN075-100MSEX, Q3 PSMN075-100MSEX, Q4 PSMN075-100MSEX, Q5 PSMN075-100MSEX, Q6 PSMN075-100MSEX, Q7 PSMN075-100MSEX, Q8 PSMN075-100MSEX, Q9 PSMN075-100MSEX, T1 PE-68386NL, U3 LT4295IUFD#PBF, U4 LT4321HUF#PBF, U5 NCP1117ST33T3G, U9 AP62250Z6

Commit message: BOM Cleanup and matching for JLCPCB, downstream edits to Schematic and Board. Added backup files to .gitignore.
Parts:
- C15, C20, C44: Comment 10u 10V 20% -> C77000 10V 10uF 20% 0402 Capacitor; PART-NUMBER GRM155R61A106ME11J -> C77000
- C16, C40: Comment 0.047u 100V 20% -> C5186810 100V 0.047uF 10% 0805 Capacitor; PART-NUMBER 08051C473K4Z2A -> C5186810
- C17, C58: Comment 0.1u 10V 20% -> C1525 16V 0.1uF 10% 0402 Capacitor; PART-NUMBER 0201ZD104KAT2A -> C1525; Rating 10V -> 16V
- C18: Comment 220p 25V 20% -> C2897613 50V 220pF 10% 0603 Capacitor; PART-NUMBER KGM15ACG1E221JT -> C2897613; Rating 25V -> 50V
- C19: Comment 3300p 25V 20% -> C5182463 50V 3300pF 10% 0603 Capacitor; PART-NUMBER KGM15AR71E332KT -> C5182463; Rating 25V -> 50V
- C41: Comment 10u 100V 20% -> C72482 100V 10uF 10% Aluminum Electrolytic Capacitors - SMD; PART-NUMBER AEK0608100M100R -> C72482; Packaging Aluminum Electrolytic Capacitors - SMD -> (none)
- C42: Comment 2.2u 100V 20% -> C6119935 100V 2.2uF 10% 0805 Capacitor; PART-NUMBER GRM21BD72A225ME01K -> C6119935
- C43, C49: Comment 2200p 2kV 20% -> C41018 2kV 2200pF 10% 1206 Capacitor; PART-NUMBER 1206GC222KAT1A -> C41018
- C45: Comment 100p 630V 20% -> C967584 1kV 100pF 5% 0805 Capacitor; PART-NUMBER GRM21A5C2J101JWA1D -> C967584; Rating 630V -> 1kV
- C46, C47, C57: Comment 10u 25V 20% -> C96446 25V 10uF 20% 0603 Capacitor; PART-NUMBER CM105X5R106M25AT -> C96446
- C48: Comment 33u 25V 20% -> C342307 25V 33uF 20% 1206 Capacitor; PART-NUMBER C3216X5R1E336M160AC -> C342307
- C50: Comment 470p 25V 20% -> C1620 50V 470pF 10% 0603 Capacitor; PART-NUMBER 06033A471KAT2A -> C1620; Rating 25V -> 50V
- C51, C52: Comment 1u 25V 20% -> C1518208 50V 1uF 10% 0402 Capacitor; PART-NUMBER TMK105BJ105MV-F -> C1518208; Rating 25V -> 50V
- C54: Comment 2200p 25V 20% -> C915853 50V 2200pF 10% 0402 Capacitor; PART-NUMBER GRM15XR71E222KA86D -> C915853; Rating 25V -> 50V
- C55: Comment 0.01u 100V 20% -> C7503490 100V 0.01uF 10% 0805 Capacitor; PART-NUMBER KAM21BR72A103KM -> C7503490
- C59, C60: Comment 22u 10V 20% -> C45783 25V 22uF 20% 0805 Capacitor; PART-NUMBER LMK212BBJ226MG-T -> C45783; Rating 10V -> 25V
- D1: Comment SMAJ24A -> C10769 SMAJ24A 10.3A 38.9V 26.7V 24V; PART-NUMBER SMAJ24A -> C10769; Packaging (none) -> DO-214AC
- D4: PART-NUMBER PTVS58VP1UTP -> (none)
- D5: value BAS19LT1G -> BAS21_R1_00001; Comment BAS19LT1G -> BAS21_R1_00001; PART-NUMBER BAS19LT1G -> C391392
- D6: Comment BAT54W -> C5186013 BAT54W; PART-NUMBER BAT54W -> C5186013
- D7: PART-NUMBER BAT46W-E3-18 -> (none)
- L1: Comment DO1608C-103 -> DO1608C-103MLC Power Inductors - SMD 10uH Shld 20% 1.5A 160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; PART-NUMBER DO1608C-103 -> (none)
- L3: PART-NUMBER DO1608C-104 -> (none)
- L4: Comment DO1813P-181HC -> DO1813P-181HC General Purpose Inductor, 0.18uH, 20%, 1 Elem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; PART-NUMBER DO1813P-181HC -> (none)
- L5: PART-NUMBER CIGT201610EH2R2MNE -> (none)
- Q1, Q2, Q3, Q4, Q5, Q6, Q7, Q8, Q9: Comment PSMN075-100MSEX -> C478016 PSMN075-100MSEX; PART-NUMBER PSMN075-100MSEX -> C478016
- Q10: PART-NUMBER FMMT723QTA -> (none)
- Q11: PART-NUMBER BSZ900N20NS3GATMA1 -> (none)
- Q12: Comment TPN1600ANH -> TPN1600ANH,L1Q; PART-NUMBER TPN1600ANH -> (none)
- Q13: Comment MMBT3906 -> C7420354 MMBT3906; PART-NUMBER MMBT3906 -> C7420354; Packaging (none) -> SOT-23
- Q14: Comment MMBT3904 -> C7420353 MMBT3904; PART-NUMBER MMBT3904 -> C7420353; Packaging (none) -> SOT-23
- R10: footprint Capacitor_SMD:C_0603_1608Metric -> Resistor_SMD:R_0603_1608Metric; Comment 26.1k 1% -> C23356 100mW Thick Film Resistors 75V 26.1kΩ 1% 0603 Resist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; PART-NUMBER CRCW060326K1FKTA -> C23356
- R21: footprint Capacitor_SMD:C_0603_1608Metric -> Resistor_SMD:R_0603_1608Metric; Comment 8.2 1% -> C23247 100mW Thick Film Resistors 75V 8.2Ω 1% 0603 Resistor; PART-NUMBER CRCW06038R20FKEAHP -> C23247
- R22: footprint Capacitor_SMD:C_0603_1608Metric -> Resistor_SMD:R_0603_1608Metric; Comment 3.3k 1% -> C22978 100mW Thick Film Resistors 75V 3.3kΩ 1% 0603 Resistor; PART-NUMBER ERJ-3GEYJ332V -> C22978
- R23: footprint Capacitor_SMD:C_0603_1608Metric -> Resistor_SMD:R_0603_1608Metric; Comment 20 1% -> C22950 100mW Thick Film Resistors 75V 20Ω 1% 0603 Resistor; PART-NUMBER CR0603-JW-200ELF -> C22950
- R24: footprint Capacitor_SMD:C_0603_1608Metric -> Resistor_SMD:R_0603_1608Metric; Comment 6.65k 1% -> C3016441 100mW Thick Film Resistors 75V 6.65kΩ 1% 0603 Resi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; PART-NUMBER CRCW06036K65FKTA -> C3016441
- R25: footprint Capacitor_SMD:C_0603_1608Metric -> Resistor_SMD:R_0603_1608Metric; Comment 2k 1% -> C22975 100mW Thick Film Resistors 75V 2kΩ 1% 0603 Resistor; PART-NUMBER RT0603FRE102KL -> C22975
- R26: footprint Capacitor_SMD:C_0805_2012Metric -> Resistor_SMD:R_0805_2012Metric; Comment 100 1/2W 5% -> C441975 500mW Thick Film Resistors 100Ω 5% 0805 Resistor; PART-NUMBER CRCW0805100RFKEAHP -> C441975
- R27: footprint LED_SMD:LED_0805_2012Metric -> Resistor_SMD:R_0805_2012Metric; Comment 25m 1/4W 5% -> C2767472 250mW Thick Film Resistors 25mΩ 5% 0805 Resistor; PART-NUMBER WSL0805R0250FEA18 -> C2767472; Packaging (none) -> 0805
- R28: footprint Capacitor_SMD:C_0805_2012Metric -> Resistor_SMD:R_1210_3225Metric; Comment 11 1/2W 5% -> C422425 1/2W Thick Film Resistors 11Ω 1% 1210 Resistor; PART-NUMBER ERJ-P06J110V -> C422425; Packaging 0805 -> 1210
- R29: footprint Capacitor_SMD:C_0603_1608Metric -> Resistor_SMD:R_0603_1608Metric; Comment 15 1% -> C22810 100mW Thick Film Resistors 75V 15Ω 1% 0603 Resistor; PART-NUMBER CRCW060315R0FKEAHP -> C22810
- R30: footprint Capacitor_SMD:C_0603_1608Metric -> Resistor_SMD:R_0603_1608Metric; Comment 100 1% -> C22775 100mW Thick Film Resistors 75V 100Ω 1% 0603 Resistor; PART-NUMBER CRCW0603100RFKEAHP -> C22775
- R31, R33: footprint Capacitor_SMD:C_0402_1005Metric -> Resistor_SMD:R_0402_1005Metric; Comment 10k 1% -> C60490 62.5mW Thick Film Resistors 50V 10kΩ 1% 0402 Resistor; PART-NUMBER CRCW040210K0FKEDC -> C60490
- R32: footprint Capacitor_SMD:C_0402_1005Metric -> Resistor_SMD:R_0402_1005Metric; Comment 52.3k 1% -> C26982 62.5mW Thick Film Resistors 50V 52.3kΩ 1% 0402 Resis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; PART-NUMBER ERJ-2RKF5232X -> C26982
- R34: footprint Capacitor_SMD:C_0603_1608Metric -> Resistor_SMD:R_0603_1608Metric; Comment 1k 1% -> C21190 100mW Thick Film Resistors 75V 1kΩ 1% 0603 Resistor; PART-NUMBER ERA-3AED102V -> C21190
- R6: footprint Capacitor_SMD:C_0603_1608Metric -> Resistor_SMD:R_0603_1608Metric; Comment 37.4 1% -> C25195 100mW Thick Film Resistors 75V 37.4Ω 1% 0603 Resistor; PART-NUMBER CRCW060337R4FKEA -> C25195
- R7: footprint Capacitor_SMD:C_0603_1608Metric -> Resistor_SMD:R_0603_1608Metric; Comment 7.5k 1% -> C23234 100mW Thick Film Resistors 75V 7.5kΩ 1% 0603 Resistor; PART-NUMBER CR0603-FX-7501ELF -> C23234
- R9: footprint Capacitor_SMD:C_0603_1608Metric -> Resistor_SMD:R_0603_1608Metric; Comment 107k 1% -> C14889 100mW Thick Film Resistors 75V 107kΩ 1% 0603 Resistor; PART-NUMBER AC0603FR-07107KL -> C14889

Commit message: BOM Finalization, board cleanup.
Parts:
- D4: value PTVS58VP1UTP -> SMF58A; footprint Diode_SMD:D_SOD-128 -> Diode_SMD:D_SOD-123; symbol Diode:PTVS26VZ1USK -> Diode:Z3SMCxxx; Comment PTVS58VP1UTP -> C435457 SMF58A; PART-NUMBER (none) -> C435457; Packaging SOD-128 -> SOD-123
- D5: Comment BAS21_R1_00001 -> C391392 BAS21_R1_00001
- D7: value BAT46W-E3-18 -> BAT46W; Comment BAT46W-E3-18 -> C5805641 BAT46W; PART-NUMBER (none) -> C5805641
- L1: footprint Custom:DO1608C -> FCH5030-100M; Comment DO1608C-103MLC Power Inductors - SMD 10uH Shld 20% 1.5A 160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 -> C20415529 FCH5030-100M; PART-NUMBER (none) -> C20415529
- L3: footprint Custom:DO1608C -> Custom:AABG05A20M101; Comment DO1608C-104 -> C5119206 AABG05A20M101; PART-NUMBER (none) -> C5119206
- L4: footprint DO1813P-181HC -> Inductor_SMD:L_0603_1608Metric; Comment DO1813P-181HC General Purpose Inductor, 0.18uH, 20%, 1 Elem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 -> C251952 LCF0603-R18J-T 1.1A 180nH ±5% SMD Power Inductors R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; PART-NUMBER (none) -> C251952; Packaging (none) -> 0603; Rating (none) -> 1.1A
- L5: Comment CIGT201610EH2R2MNE -> C337891 1.7A 2.2uH ±20% 140mΩ 0806 Inductors (SMD); PART-NUMBER (none) -> C337891
- Q10: Comment FMMT723QTA -> C5249004 FMMT723QTA; PART-NUMBER (none) -> C5249004
- Q11: Comment BSZ900N20NS3GATMA1 -> C3279283 BSZ900N20NS3GATMA1; PART-NUMBER (none) -> C3279283
- Q12: Comment TPN1600ANH,L1Q -> C24363903 TPN1600ANH,L1Q; PART-NUMBER (none) -> C24363903
- T1: Comment PE-68386NL -> C581397 PE-68386NL; PART-NUMBER PE-68386NL -> C581397
- TR1: Comment 750316115 -> C24363903 750316115; PART-NUMBER 750316115 -> C24363903
- U3: Comment LT4295IUFD#PBF -> C672449 LT4295IUFD#PBF; PART-NUMBER LT4295IUFD#PBF -> C672449
- U4: Comment LT4321HUF#PBF -> C672474 LT4321HUF#PBF; PART-NUMBER LT4321HUF#PBF -> C672474
- U5: Comment NCP1117ST33T3G -> C26537 NCP1117ST33T3G; PART-NUMBER NCP1117ST33T3G -> C26537
- U9: Comment AP62250Z6 -> C5290220 AP62250Z6; PART-NUMBER AP62250Z6 -> C5290220
Changed lines of the file:
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@@
 			)
 		)
-		(property "Value" "BAT46W-E3-18"
+		(property "Value" "BAT46W"
 			(at 361.95 131.7624 90)
 			(effects
@@
 			)
 		)
-		(property "Datasheet" "BAT46W-E3-18"
+		(property "Datasheet" "BAT46W"
 			(at 359.41 130.81 0)
 			(effects
@@
 			)
 		)
-		(property "PART-NUMBER" ""
+		(property "PART-NUMBER" "C5805641"
 			(at 359.41 130.81 90)
 			(effects
@@
 			)
 		)
-		(property "Comment" "BAT46W-E3-18"
+		(property "Comment" "C5805641 BAT46W"
 			(at 359.41 130.81 0)
 			(effects
@@
 			)
 		)
-		(property "PART-NUMBER" "AP62250Z6"
+		(property "PART-NUMBER" "C5290220"
 			(at 336.55 184.15 0)
 			(effects
@@
 			)
 		)
-		(property "Comment" "AP62250Z6"
+		(property "Comment" "C5290220 AP62250Z6"
 			(at 336.55 184.15 0)
 			(effects
@@
 			)
 		)
-		(property "Comment" "BAS21_R1_00001"
+		(property "Comment" "C391392 BAS21_R1_00001"
 			(at 222.25 81.28 0)
 			(effects
@@
 			)
 		)
-		(property "PART-NUMBER" ""
+		(property "PART-NUMBER" "C24363903"
 			(at 344.17 78.74 0)
 			(effects
@@
 			)
 		)
-		(property "Comment" "TPN1600ANH,L1Q"
+		(property "Comment" "C24363903 TPN1600ANH,L1Q"
 			(at 344.17 78.74 0)
 			(effects
@@
 			)
 		)
-		(property "Footprint" "Custom:DO1608C"
+		(property "Footprint" "FCH5030-100M"
 			(at 203.2 45.72 0)
 			(effects
@@
 			)
 		)
-		(property "Datasheet" "DO1608C-104"
+		(property "Datasheet" "FCH5030-100M"
 			(at 203.2 45.72 0)
 			(effects
@@
 			)
 		)
-		(property "PART-NUMBER" ""
+		(property "PART-NUMBER" "C20415529"
 			(at 203.2 45.72 0)
 			(effects
@@
 			)
 		)
-		(property "Comment" "DO1608C-103MLC Power Inductors - SMD 10uH Shld 20% 1.5A 160mOhms "
+		(property "Comment" "C20415529 FCH5030-100M"
 			(at 203.2 45.72 0)
 			(effects
@@
 			)
 		)
-		(property "PART-NUMBER" ""
+		(property "PART-NUMBER" "C5249004"
 			(at 227.33 68.58 0)
 			(effects
@@
 			)
 		)
-		(property "Comment" "FMMT723QTA"
+		(property "Comment" "C5249004 FMMT723QTA"
 			(at 227.33 68.58 0)
 			(effects
@@
 			)
 		)
-		(property "PART-NUMBER" "LT4321HUF#PBF"
+		(property "PART-NUMBER" "C672474"
 			(at 46.99 196.85 0)
 			(effects
@@
 			)
 		)
-		(property "Comment" "LT4321HUF#PBF"
+		(property "Comment" "C672474 LT4321HUF#PBF"
 			(at 46.99 196.85 0)
 			(effects
@@
 			)
 		)
-		(property "PART-NUMBER" ""
+		(property "PART-NUMBER" "C3279283"
 			(at 289.56 97.79 0)
 			(effects
@@
 			)
 		)
-		(property "Comment" "BSZ900N20NS3GATMA1"
+		(property "Comment" "C3279283 BSZ900N20NS3GATMA1"
 			(at 289.56 97.79 0)
 			(effects
@@
 		(on_board yes)
 		(dnp no)
-		(fields_autoplaced yes)
 		(property "Reference" "L4"
 			(at 365.76 48.26 90)
@@
 			)
 		)
-		(property "Footprint" "DO1813P-181HC"
+		(property "Footprint" "Inductor_SMD:L_0603_1608Metric"
 			(at 365.76 53.34 0)
 			(effects
@@
 			)
 		)
-		(property "Packaging" ""
+		(property "Packaging" "0603"
 			(at 365.76 53.34 90)
 			(effects
@@
 			)
 		)
-		(property "PART-NUMBER" ""
+		(property "PART-NUMBER" "C251952"
 			(at 365.76 53.34 90)
 			(effects
@@
 			)
 		)
-		(property "Comment" "DO1813P-181HC General Purpose Inductor, 0.18uH, 20%, 1 Element, SMD, 3524"
+		(property "Comment" "C251952 LCF0603-R18J-T 1.1A 180nH ±5% SMD Power Inductors ROHS"
 			(at 365.76 53.34 0)
 			(effects
@@
 			)
 		)
+		(property "Rating" "1.1A "
+			(at 371.348 50.8 90)
+			(effects
+				(font
+					(size 1.27 1.27)
+				)
+			)
+		)
 		(pin "1"
 		)
@@
 			)
 		)
-		(property "PART-NUMBER" "LT4295IUFD#PBF"
+		(property "PART-NUMBER" "C672449"
 			(at 212.09 119.38 0)
 			(effects
@@
 			)
 		)
-		(property "Comment" "LT4295IUFD#PBF"
+		(property "Comment" "C672449 LT4295IUFD#PBF"
 			(at 212.09 119.38 0)
 			(effects
@@
 			)
 		)
-		(property "Footprint" "Custom:DO1608C"
+		(property "Footprint" "Custom:AABG05A20M101"
 			(at 233.68 77.47 0)
 			(effects
@@
 			)
 		)
-		(property "Datasheet" "DO1608C-104"
+		(property "Datasheet" "AABG05A20M101"
 			(at 233.68 77.47 0)
 			(effects
@@
 			)
 		)
-		(property "PART-NUMBER" ""
+		(property "PART-NUMBER" "C5119206"
 			(at 233.68 77.47 90)
 			(effects
@@
 			)
 		)
-		(property "Comment" "DO1608C-104"
+		(property "Comment" "C5119206 AABG05A20M101"
 			(at 233.68 77.47 0)
 			(effects
@@
 			)
 		)
-		(property "PART-NUMBER" "PE-68386NL"
+		(property "PART-NUMBER" "C581397"
 			(at 311.15 130.81 0)
 			(effects
@@
 			)
 		)
-		(property "Comment" "PE-68386NL"
+		(property "Comment" "C581397 PE-68386NL"
 			(at 311.15 130.81 0)
 			(effects
@@
 	)
 	(symbol
-		(lib_id "Diode:PTVS26VZ1USK")
+		(lib_id "Diode:Z3SMCxxx")
 		(at 152.4 137.16 270)
 		(unit 1)
@@
 			)
 		)
-		(property "Value" "PTVS58VP1UTP"
+		(property "Value" "SMF58A"
 			(at 154.94 138.4299 90)
 			(effects
@@
 			)
 		)
-		(property "Footprint" "Diode_SMD:D_SOD-128"
+		(property "Footprint" "Diode_SMD:D_SOD-123"
 			(at 147.955 137.16 0)
 			(effects
@@
 			)
 		)
-		(property "Datasheet" "PTVS58VP1UTP"
+		(property "Datasheet" ""
 			(at 152.4 137.16 0)
 			(effects
@@
 			)
 		)
-		(property "PART-NUMBER" ""
+		(property "PART-NUMBER" "C435457"
 			(at 152.4 137.16 90)
 			(effects
@@
 			)
 		)
-		(property "Packaging" "SOD-128"
+		(property "Packaging" "SOD-123"
 			(at 152.4 137.16 90)
 			(effects
@@
 			)
 		)
-		(property "Comment" "PTVS58VP1UTP"
+		(property "Comment" "C435457 SMF58A"
 			(at 152.4 137.16 0)
 			(effects
@@
 			)
 		)
-		(property "PART-NUMBER" "NCP1117ST33T3G"
+		(property "PART-NUMBER" "C26537"
 			(at 347.98 231.14 0)
 			(effects
@@
 			)
 		)
-		(property "Comment" "NCP1117ST33T3G"
+		(property "Comment" "C26537 NCP1117ST33T3G"
 			(at 347.98 231.14 0)
 			(effects
@@
 			)
 		)
-		(property "PART-NUMBER" "750316115"
+		(property "PART-NUMBER" "C24363903"
 			(at 311.15 58.42 0)
 			(effects
@@
 			)
 		)
-		(property "Comment" "750316115"
+		(property "Comment" "C24363903 750316115"
 			(at 311.15 58.42 0)
 			(effects
@@
 			)
 		)
-		(property "Datasheet" "CIGT201610EH2R2MNE"
+		(property "Datasheet" "DFE201610E-2R2M=P2"
 			(at 368.3 181.61 0)
 			(effects
@@
 			)
 		)
-		(property "PART-NUMBER" ""
+		(property "PART-NUMBER" "C337891 "
 			(at 368.3 181.61 90)
 			(effects
@@
 			)
 		)
-		(property "Comment" "CIGT201610EH2R2MNE"
+		(property "Comment" "C337891 1.7A 2.2uH ±20% 140mΩ 0806 Inductors (SMD)"
 			(at 368.3 181.61 0)
 			(effects
