File: uC.kicad_sch (KiCad schematic)
At the start: 56 parts, among them U1 RP2040, U2 W25Q128JVS, U6 LAN9500A-ABZJ-TR, U7 93AA46AT-I/OT, Y1 ABM8-272-T3, Y2 ABM8G-25.000MHZ-4Y-T3

Commit message: BOM Cleanup and matching for JLCPCB, downstream edits to Schematic and Board. Added backup files to .gitignore.
Parts:
- C1, C4: Comment 1u 25V 20% -> C1518208 50V 1uF 10% 0402 Capacitor; PART-NUMBER TMK105BJ105MV-F -> C1518208; Rating 25V -> 50V
- C10, C11, C12, C2, C23, C24, C25, C26, C27, C28, C29, C3, C5, C6, C7, C8, C9: Comment 0.1u 10V 20% -> C1525 16V 0.1uF 10% 0402 Capacitor; PART-NUMBER 0201ZD104KAT2A -> C1525; Rating 10V -> 16V
- C13, C14: Comment 15p 10V 20% -> C1548 50V 15pF 5% 0402 Capacitor; PART-NUMBER VJ0402A150KXQCW1BC -> C1548; Rating 10V -> 50V
- C21, C22: Comment 10p 10V 20% -> C1545 50V 10pF 5% 0402 Capacitor; PART-NUMBER C0402C100J8GACTU -> C1545
- C30, C31, C32, C33, C34, C35: Comment 4700p 10V 20% -> C7503510 10V 4700pF 10% 0402 Capacitor; PART-NUMBER LMK105SD472JV-F -> C7503510
- C36, C37, C38: Comment 1500p 10V 20% -> C284989 50V 1500pF 10% 0402 Capacitor; PART-NUMBER 885012205007 -> C284989; Rating 10V -> 50V
- D2, D3: PART-NUMBER LTST-C193TBKT-5A -> (none)
- FB1, FB2, FB3: Comment BLM21AG121SN1D -> C88990 100mΩ ±25% 120Ω@100MHz 0805 Ferrite Beads; PART-NUMBER BLM21AG121SN1D -> C88990
- R1, R2: footprint Capacitor_SMD:C_0402_1005Metric -> Resistor_SMD:R_0402_1005Metric; Comment 27.4 1% -> C284479 62.5mW Thick Film Resistors 50V 27.4Ω 1% 0402 Resis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; PART-NUMBER RT0402BRE0727R4L -> C284479
- R13, R14, R19: footprint Capacitor_SMD:C_0402_1005Metric -> Resistor_SMD:R_0402_1005Metric; Comment 12k 1% -> C102781 62.5mW Thick Film Resistors 50V 12kΩ 1% 0402 Resist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; PART-NUMBER MCS04020D1202BE000 -> C102781
- R15, R17: footprint Capacitor_SMD:C_0402_1005Metric -> Resistor_SMD:R_0402_1005Metric; Comment 330 1% -> C25104 62.5mW Thick Film Resistors 50V 330Ω 1% 0402 Resistor; PART-NUMBER CR0402-FX-3300GLF -> C25104
- R16: footprint Capacitor_SMD:C_0402_1005Metric -> Resistor_SMD:R_0402_1005Metric; Comment 0 1% -> C17168 62.5mW Thick Film Resistors 50V 0Ω 1% 0402 Resistor; PART-NUMBER CRCW04020000Z0EEHP -> C17168
- R18, R3, R5: footprint Capacitor_SMD:C_0402_1005Metric -> Resistor_SMD:R_0402_1005Metric; Comment 1k 1% -> C106235 62.5mW Thick Film Resistors 50V 1kΩ 1% 0402 Resistor; PART-NUMBER CRT0402AFY-1001GLF -> C106235
- R20: footprint Capacitor_SMD:C_0402_1005Metric -> Resistor_SMD:R_0402_1005Metric; Comment 10k 1% -> C60490 62.5mW Thick Film Resistors 50V 10kΩ 1% 0402 Resistor; PART-NUMBER CRCW040210K0FKEDC -> C60490
- R4: footprint Diode_SMD:D_0402_1005Metric -> Resistor_SMD:R_0402_1005Metric; Comment 0 1% -> C17168 62.5mW Thick Film Resistors 50V 0Ω 1% 0402 Resistor; PART-NUMBER CRCW04020000Z0EEHP -> C17168
- U1: Comment RP2040 -> C2040 RP2040; PART-NUMBER RP2040 -> C2040

Commit message: BOM Finalization, board cleanup.
Parts:
- U2: Comment W25Q128JVS -> C97521 W25Q128JVS; PART-NUMBER W25Q128JVS -> C97521
- U6: Comment LAN9500A-ABZJ-TR -> C2651877 LAN9500A-ABZJ-TR; PART-NUMBER LAN9500A-ABZJ-TR -> C2651877
- U7: Comment 93AA46AT-I/OT -> C145736 93AA46AT-I/OT; PART-NUMBER 93AA46AT-I/OT -> C145736
- Y1: Comment ABM8-272-T3 -> C20625731 ABM8-272-T3; PART-NUMBER ABM8-272-T3 -> C20625731
- Y2: Comment ABM8G-25.000MHZ-4Y-T3 -> C596914 ABM8G-25.000MHZ-4Y-T3; PART-NUMBER ABM8G-25.000MHZ-4Y-T3 -> C596914
Changed lines of the file:
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@@
 			)
 		)
-		(property "PART-NUMBER" "W25Q128JVS"
+		(property "PART-NUMBER" "C97521"
 			(at 382.27 226.06 0)
 			(effects
@@
 			)
 		)
-		(property "Comment" "W25Q128JVS"
+		(property "Comment" "C97521 W25Q128JVS"
 			(at 382.27 226.06 0)
 			(effects
@@
 			)
 		)
-		(property "PART-NUMBER" "ABM8-272-T3"
+		(property "PART-NUMBER" "C20625731"
 			(at 288.29 220.98 90)
 			(effects
@@
 			)
 		)
-		(property "Comment" "ABM8-272-T3"
+		(property "Comment" "C20625731 ABM8-272-T3"
 			(at 288.29 220.98 0)
 			(effects
@@
 			)
 		)
-		(property "PART-NUMBER" "93AA46AT-I/OT"
+		(property "PART-NUMBER" "C145736"
 			(at 198.12 262.89 0)
 			(effects
@@
 			)
 		)
-		(property "Comment" "93AA46AT-I/OT"
+		(property "Comment" "C145736 93AA46AT-I/OT"
 			(at 198.12 262.89 0)
 			(effects
@@
 			)
 		)
-		(property "PART-NUMBER" "ABM8G-25.000MHZ-4Y-T3"
+		(property "PART-NUMBER" "C596914"
 			(at 195.58 224.79 90)
 			(effects
@@
 			)
 		)
-		(property "Comment" "ABM8G-25.000MHZ-4Y-T3"
+		(property "Comment" "C596914 ABM8G-25.000MHZ-4Y-T3"
 			(at 195.58 224.79 0)
 			(effects
@@
 			)
 		)
-		(property "PART-NUMBER" "LAN9500A-ABZJ-TR"
+		(property "PART-NUMBER" "C2651877"
 			(at 58.42 130.81 0)
 			(effects
@@
 			)
 		)
-		(property "Comment" "LAN9500A-ABZJ-TR"
+		(property "Comment" "C2651877 LAN9500A-ABZJ-TR"
 			(at 58.42 130.81 0)
 			(effects
